Commit message: changed link name to map

File: src/joint_description/urdf/joint_model.urdf (robot description, URDF)
Before this commit: robot joint_model, 5 links, 4 joints
Links:
- removed link world
- added link map
Joints:
- joint base_joint: parent world -> map

Commit message: Minor changes

File: src/joint_description/urdf/joint_model.urdf (robot description, URDF)
Before this commit: robot joint_model, 5 links, 4 joints
Links:
- removed link map
- added link world

Commit message: Added config file

File: src/joint_description/urdf/joint_model.urdf (robot description, URDF)
Before this commit: robot joint_model, 2 links, 0 joints
Links:
- removed link base_link

Commit message: Minor changes

File: src/joint_description/urdf/joint_model.urdf (robot description, URDF)
Before this commit: robot joint_model, 1 links, 0 joints
Links:
- added link base_link
